Commit message: [CAM] Added cam on front of the submarine

File: hrov_description/urdf/sensors.xacro (robot description, xacro)
@@ -33,5 +33,5 @@
   <!-- Mount a camera  -->
   <xacro:default_camera namespace="${namespace}" parent_link="${namespace}/base_link" suffix="">
-    <origin xyz="0 0 -1" rpy="0 0 0"/>
+    <origin xyz="2.7658 0 -0.0830" rpy="0 0 0"/>
   </xacro:default_camera>
 </robot>
