Commit message: [FINS] Added 3d model for fins, ans setup, works perfectly

File: hrov_description/urdf/actuators.xacro (robot description, xacro)
@@ -21,11 +21,11 @@
   </xacro:thruster_macro-->
     <!-- Instantiate fins, if necessary -->
-    <!--xacro:fin_macro namespace="${namespace}" fin_id="0">
-      <origin xyz="0 0 0" rpy="0 0 0" />
+    <xacro:fin_macro namespace="${namespace}" fin_id="0" mesh_filename="${fin_mesh_file}">
+      <origin xyz="-2.75873 0.757596 0.020071" rpy="${0.5 * pi} 0 0" />
     </xacro:fin_macro>
-    <xacro:fin_macro namespace="${namespace}" fin_id="1">
-      <origin xyz="0 0 0" rpy="0 0 0" />
+    <xacro:fin_macro namespace="${namespace}" fin_id="1" mesh_filename="${fin_mesh_file}">
+      <origin xyz="-2.75873 -0.757596 0.020071" rpy="${0.5 * pi} 0 0" />
     </xacro:fin_macro>
-    <xacro:fin_macro namespace="${namespace}" fin_id="2">
+    <!--xacro:fin_macro namespace="${namespace}" fin_id="2">
       <origin xyz="0 0 0" rpy="0 0 0" />
     </xacro:fin_macro>

File: hrov_description/urdf/sensors.xacro (robot description, xacro)
@@ -33,5 +33,5 @@
   <!-- Mount a camera  -->
   <xacro:default_camera namespace="${namespace}" parent_link="${namespace}/base_link" suffix="">
-    <origin xyz="0 0 0" rpy="0 0 0"/>
+    <origin xyz="0 0 -1" rpy="0 0 0"/>
   </xacro:default_camera>
 </robot>

File: hrov_description/urdf/snippets.xacro (robot description, xacro)
@@ -165,21 +165,23 @@
   <!-- A separate mesh for the fin should be stored in the meshes folder -->
   <xacro:property name="fin_mesh_file" value="file://$(find hrov_description)/meshes/fin.dae"/>
-  <!-- Fin joint limits  -->
-  <xacro:property name="fin_min_joint_limit" value="${0.0 * d2r}"/>
-  <xacro:property name="fin_max_joint_limit" value="${0.0 * d2r}"/>
-  <xacro:macro name="fin_macro" params="namespace fin_id *origin mesh_filename">
-    <xacro:fin_quadratic_macro
-      namespace="${namespace}"
-      parent_link="${namespace}/base_link"
-      fin_id="${fin_id}"
-      min_joint_limit="${-90.0 * d2r}"
-      max_joint_limit="${90.0 * d2r}"
-      mesh_filename="${mesh_filename}"
-      fin_dynamics_time_constant="0.2"
-      lift_constant="${0.5 * fin_rho * fin_area * fin_lift_coefficient}"
-      drag_constant="${0.5 * fin_rho * fin_area * fin_drag_coefficient}"
-      current_velocity_topic="current_velocity">
-      <xacro:insert_block name="origin"/>
-    </xacro:fin_quadratic_macro>
-</xacro:macro>
+    <!-- Fin properties -->
+    <xacro:property name="fin_area" value="0.0064"/>
+    <xacro:property name="fin_rho" value="1028"/>
+    <xacro:property name="fin_lift_coefficient" value="3.0"/>
+    <xacro:property name="fin_drag_coefficient" value="1.98"/>
+    <xacro:macro name="fin_macro" params="namespace fin_id *origin mesh_filename">
+        <xacro:fin_quadratic_macro
+          namespace="${namespace}"
+          parent_link="${namespace}/base_link"
+          fin_id="${fin_id}"
+          min_joint_limit="${-90.0 * d2r}"
+          max_joint_limit="${90.0 * d2r}"
+          mesh_filename="${mesh_filename}"
+          fin_dynamics_time_constant="0.2"
+          lift_constant="${0.5 * fin_rho * fin_area * fin_lift_coefficient}"
+          drag_constant="${0.5 * fin_rho * fin_area * fin_drag_coefficient}"
+          current_velocity_topic="current_velocity">
+          <xacro:insert_block name="origin"/>
+        </xacro:fin_quadratic_macro>
+    </xacro:macro>
 </robot>

Commit message: [THRUSTERS] Now good angle

File: hrov_description/urdf/actuators.xacro (robot description, xacro)
@@ -9,8 +9,8 @@
     -->
     <xacro:thruster_macro robot_namespace="${namespace}" thruster_id="0">
-        <origin xyz="-2.57 0.76 0.024" rpy="0 0 ${pi}" />
+        <origin xyz="-2.57 0.76 0.024" rpy="0 0 0" />
     </xacro:thruster_macro>
     <xacro:thruster_macro robot_namespace="${namespace}" thruster_id="1">
-        <origin xyz="-2.57 -0.76 0.024" rpy="0 0 ${pi}" />
+        <origin xyz="-2.57 -0.76 0.024" rpy="0 0 0" />
     </xacro:thruster_macro>
     <!--xacro:thruster_macro robot_namespace="${namespace}" thruster_id="1">
